File: kicad/rak3172_board/RAK proto board.kicad_pcb (KiCad board)
At the start: 2 copper layers, 51 x 36 mm, 39 parts, among them J1 JTAG, J4 Groove AIN0 AIN1, J5 Groove AIN2 AIN3

Commit message: Updated schematic and pcb
Parts:
- removed the D1 at (176.3, 59.1)
- removed R2: 1K, Resistor_SMD:R_0603_1608Metric_Pad0.98x0.95mm_HandSolder
- D1: renamed from D2; footprint Diode_SMD:D_1206_3216Metric_Pad1.42x1.75mm_HandSolder -> Diode_SMD:D_0603_1608Metric
- J2: renamed from UART2 AT
- J7: renamed from Battery; moved to B.Cu
- moved R1 1.78 mm to (172.5, 61.2)
- moved D1 1.65 mm to (176.3, 61.2)
- moved C3 0.43 mm to (156.3, 52.8)
- moved C2 0.35 mm to (159.0, 52.3)
- turned J7 to 0 degrees
- renumbered UART1 to J3, I2C to J6, KPS to Q1, SWITCH to SW1, RAK3172 to U1, ADS1115 to U2, BME680 to U3, LIS2DH12 to U4
Routing:
- net D0: track 31.1 -> 0.77 mm, vias 2 -> 0
- net Net-(D1-A) (its old number): track 2.10 -> 0.00 mm
- net +3V3: track 151.3 -> 149.3 mm
- net D1: track 40.5 -> 38.5 mm
- net RST: track 27.5 -> 28.5 mm
- net SDA: track 93.4 -> 92.5 mm
- net SCL: track 86.8 -> 86.2 mm
- net D2: track 26.4 -> 27.0 mm
- net GND: track 45.1 -> 45.0 mm, vias 18 -> 17

Commit message: Ordered v1.0 on JLCPCB
Parts:
- removed the C3 at (156.3, 52.8)
- removed J2: UART2 AT, Grove 4 Pins:Grove 4 Pins
- removed J3: UART1, Grove 4 Pins:Grove 4 Pins
- removed J4: Groove AIN0 AIN1, Grove 4 Pins:Grove 4 Pins
- removed J5: Groove AIN2 AIN3, Grove 4 Pins:Grove 4 Pins
- removed J6: I2C, Grove 4 Pins:Grove 4 Pins
- removed the R6 at (161.3, 51.7)
- removed the R8 at (148.6, 57.4)
- removed U2: ADS1115IDGS, Package_SO:TSSOP-10_3x3mm_P0.5mm
- added A1/A2: Groove A1 A2, Connector_JST:JST_PH_B4B-PH-K_1x04_P2.00mm_Vertical, F.Cu at (154.3, 63.4)
- added A3/A4: Groove A3 A4, Connector_JST:JST_PH_B4B-PH-K_1x04_P2.00mm_Vertical, F.Cu at (169.1, 63.4)
- added BOOT0: SW BOOT0, Button_Switch_SMD:SW_Push_1P1T_NO_CK_KMR2, F.Cu at (156.3, 53.6)
- added C12: 1uF, Capacitor_Tantalum_SMD:CP_EIA-1608-08_AVX-J, F.Cu at (163.5, 51.1)
- added C13: 0, Capacitor_Tantalum_SMD:CP_EIA-1608-08_AVX-J, F.Cu at (143.6, 38.9)
- added DIGITAL1: DIGITAL, Connector_JST:JST_PH_B4B-PH-K_1x04_P2.00mm_Vertical, F.Cu at (178.7, 57.1)
- added G***: LOGO, RAK_Library:logo_polytech, B.Cu at (136.5, 31.6)
- added I2C1: I2C, Connector_JST:JST_PH_B4B-PH-K_1x04_P2.00mm_Vertical, F.Cu at (148.2, 30.0)
- added R10: 0, Resistor_SMD:R_0603_1608Metric_Pad0.98x0.95mm_HandSolder, F.Cu at (144.4, 35.2)
- added R11: 0, Resistor_SMD:R_0603_1608Metric_Pad0.98x0.95mm_HandSolder, F.Cu at (144.0, 41.5)
- added UART1: UART1, Connector_JST:JST_PH_B4B-PH-K_1x04_P2.00mm_Vertical, F.Cu at (163.1, 30.0)
- added UART2: UART2 AT, Connector_JST:JST_PH_B4B-PH-K_1x04_P2.00mm_Vertical, F.Cu at (178.7, 30.3)
- R9: value 0 -> 10K
- moved BATTERY1 16.1 mm to (159.7, 58.4), turned to 90 degrees
- moved R9 9.55 mm to (153.6, 56.4)
- moved C5 5.30 mm to (145.6, 56.4)
- moved R8 4.88 mm to (145.7, 58.4), turned to 180 degrees
- moved JTAG1 3.61 mm to (182.2, 46.8)
- moved C10 3.44 mm to (150.9, 57.1)
- moved C6 3.27 mm to (152.9, 59.1)
- moved C8 3.02 mm to (149.4, 59.1)
- moved LIS2DH12 2.86 mm to (172.6, 53.7)
- moved KPS-3227 2.74 mm to (146.8, 53.5), turned to -90 degrees
- moved C3 2.72 mm to (169.0, 53.6)
- moved D1 2.39 mm to (174.1, 62.3), turned to -90 degrees
- moved R6 2.15 mm to (144.8, 30.4)
- moved R7 1.96 mm to (143.2, 30.4)
- moved BME680 1.81 mm to (172.1, 41.4)
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- renumbered J7 to BATTERY1, U3 to BME680, C8 to C10, C9 to C11, C11 to C3, C12 to C4, C10 to C5, C5 to C6, C6 to C7, C4 to C8, C7 to C9, J1 to JTAG1, Q1 to KPS-3227, U4 to LIS2DH12, R11 to R2, R12 to R3, R10 to R4, R3 to R5, R4 to R6, R5 to R7, R7 to R8, U1 to RAK3172, SW1 to RST1
Connections:
- C10 pad 1: AIN1 -> A1
- C10 pad 2: AIN0 -> A0
- C11 pad 1: AIN3 -> A3
- C11 pad 2: AIN2 -> A2
- C5 pad 2: Net-(C10-Pad2) -> A4
- C6 pad 2: AIN1 -> A1
- C7 pad 2: AIN3 -> A3
- C8 pad 2: AIN0 -> A0
- C9 pad 2: AIN2 -> A2
- D1 pad 1: D1 -> D3
- KPS-3227 pad 2: Net-(C10-Pad2) -> A4
- KPS-3227 pad 4: Net-(C10-Pad2) -> A4
- LIS2DH12 pad 11: unconnected-(U4-INT_2-Pad11) -> D0
- LIS2DH12 pad 12: unconnected-(U4-INT_1-Pad12) -> D5
- R8 pad 2: Net-(C10-Pad2) -> A4
- R9 pad 1: AIN0 -> GND
- R9 pad 2: Net-(C10-Pad2) -> BOOT0
- RAK3172 pad 21: GND -> BOOT0
Routing:
- net A2: track 0.00 -> 35.4 mm
- net D0: track 0.77 -> 31.5 mm, vias 0 -> 2
- net A0: track 0.00 -> 30.7 mm
- net A4: track 0.00 -> 29.6 mm
- net A1: track 0.00 -> 28.5 mm
- net GND: track 45.0 -> 72.4 mm, vias 17 -> 13
- net D3: track 0.00 -> 27.3 mm, vias 0 -> 2
- net D5: track 0.00 -> 23.6 mm, vias 0 -> 2
- net AIN3: track 20.5 -> 0.00 mm
- net AIN0: track 19.8 -> 0.00 mm
- net AIN2: track 18.4 -> 0.00 mm
- net SCL: track 86.2 -> 68.5 mm, vias 3 -> 5
- net Net-(C10-Pad2): track 15.7 -> 0.00 mm
- net AIN1: track 14.5 -> 0.00 mm
- net SDA: track 92.5 -> 78.1 mm
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- added copper zone on F.Cu, net GND
Other:
- board size 51 x 36 mm -> 51 x 37 mm
- board text added: "RAKI2HM v1.0"
