File: kicad/rak3172_board/RAK proto board.kicad_sch (KiCad schematic)
At the start: 39 parts, among them J1 JTAG, J2 UART2 AT, J3 UART1, J4 Groove AIN0 AIN1, J5 Groove AIN2 AIN3, J6 I2C, J7 Battery, Q1 KPS-3227, U1 RAK3172, U2 ADS1115IDGS, U3 BME680, U4 LIS2DH12

Commit message: Updated schematic and pcb
Parts:
- removed D1: GREEN, Diode_SMD:D_1206_3216Metric_Pad1.42x1.75mm_HandSolder, symbol Device:LED
- removed R2: 1K, Resistor_SMD:R_0603_1608Metric_Pad0.98x0.95mm_HandSolder, symbol Device:R
- D1: renamed from D2; footprint Diode_SMD:D_1206_3216Metric_Pad1.42x1.75mm_HandSolder -> Diode_SMD:D_0603_1608Metric
Changed lines of the file:
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@@
-    (stroke (width 0) (type default))
-  )
-  (wire (pts (xy 36.83 95.25) (xy 39.37 95.25))
     (stroke (width 0) (type default))
   )
@@
     (stroke (width 0) (type default))
   )
-  (wire (pts (xy 27.94 95.25) (xy 29.21 95.25))
-    (stroke (width 0) (type default))
-  )
   (wire (pts (xy 114.3 124.46) (xy 114.3 119.38))
     (stroke (width 0) (type default))
@@
     (stroke (width 0) (type default))
   )
-  (wire (pts (xy 27.94 93.98) (xy 27.94 95.25))
-    (stroke (width 0) (type default))
-  )
   (wire (pts (xy 248.92 26.67) (xy 255.27 26.67))
     (stroke (width 0) (type default))
@@
   )
   (wire (pts (xy 107.95 38.1) (xy 111.76 38.1))
-    (stroke (width 0) (type default))
-  )
-  (wire (pts (xy 46.99 95.25) (xy 62.23 95.25))
     (stroke (width 0) (type default))
   )
@@
     (effects (font (size 1.27 1.27) (color 132 0 0 1)) (justify left top))
   )
-  (text_box "I2C"
-    (at 313.69 -10.16 0) (size 107.95 90.17)
-    (stroke (width 0) (type default) (color 132 0 0 1))
-    (fill (type none))
-    (effects (font (size 1.27 1.27) (color 132 0 0 1)) (justify left top))
-  )
   (text_box "Gas / Humidity / Temperature / Pressure Sensor"
     (at 146.05 104.14 0) (size 59.69 40.64)
@@
     (effects (font (size 1.27 1.27)) (justify left))
     (property "Intersheetrefs" "${INTERSHEET_REFS}" (at 118.4947 45.72 0)
-      (effects (font (size 1.27 1.27)) (justify left) hide)
-    )
-  )
-  (global_label "D0" (shape input) (at 62.23 95.25 0) (fields_autoplaced)
-    (effects (font (size 1.27 1.27)) (justify left))
-    (property "Intersheetrefs" "${INTERSHEET_REFS}" (at 66.9457 95.25 0)
       (effects (font (size 1.27 1.27)) (justify left) hide)
     )
@@
     )
   )
-  (symbol (lib_id "Device:LED") (at 43.18 95.25 180) (unit 1)
-    (in_bom yes) (on_board yes) (dnp no)
-    (property "Reference" "D1" (at 40.64 97.79 0)
-      (effects (font (size 1.27 1.27)))
-    )
-    (property "Value" "GREEN" (at 46.99 97.79 0)
-      (effects (font (size 1.27 1.27)))
-    )
-    (property "Footprint" "Diode_SMD:D_1206_3216Metric_Pad1.42x1.75mm_HandSolder" (at 43.18 95.25 0)
-      (effects (font (size 1.27 1.27)) hide)
-    )
-    (property "Datasheet" "~" (at 43.18 95.25 0)
-      (effects (font (size 1.27 1.27)) hide)
-    )
-    (pin "1")
-    (pin "2")
-    (instances
-      (project "RAK proto board"
-        (path "/320cfaa9-598b-4438-8ba0-f401c00f1f04"
-          (reference "D1") (unit 1)
-        )
-      )
-    )
-  )
   (symbol (lib_id "power:GND") (at 80.01 81.28 0) (unit 1)
     (in_bom yes) (on_board yes) (dnp no)
@@
   (symbol (lib_id "Device:LED") (at 43.18 86.36 180) (unit 1)
     (in_bom yes) (on_board yes) (dnp no)
-    (property "Reference" "D2" (at 40.64 88.9 0)
+    (property "Reference" "D1" (at 40.64 88.9 0)
       (effects (font (size 1.27 1.27)))
     )
@@
       (effects (font (size 1.27 1.27)))
     )
-    (property "Footprint" "Diode_SMD:D_1206_3216Metric_Pad1.42x1.75mm_HandSolder" (at 43.18 86.36 0)
+    (property "Footprint" "Diode_SMD:D_0603_1608Metric" (at 43.18 86.36 0)
       (effects (font (size 1.27 1.27)) hide)
     )
@@
       (project "RAK proto board"
         (path "/320cfaa9-598b-4438-8ba0-f401c00f1f04"
-          (reference "D2") (unit 1)
+          (reference "D1") (unit 1)
         )
       )
@@
     )
   )
-  (symbol (lib_id "power:+3V3") (at 27.94 93.98 0) (unit 1)
-    (in_bom yes) (on_board yes) (dnp no)
-    (property "Reference" "#PWR012" (at 27.94 97.79 0)
-      (effects (font (size 1.27 1.27)) hide)
-    )
-    (property "Value" "+3V3" (at 25.4 91.44 0)
-      (effects (font (size 1.27 1.27)))
-    )
-    (property "Footprint" "" (at 27.94 93.98 0)
-      (effects (font (size 1.27 1.27)) hide)
-    )
-    (property "Datasheet" "" (at 27.94 93.98 0)
-      (effects (font (size 1.27 1.27)) hide)
-    )
-    (pin "1")
-    (instances
-      (project "RAK proto board"
-        (path "/320cfaa9-598b-4438-8ba0-f401c00f1f04"
-          (reference "#PWR012") (unit 1)
-        )
-      )
-    )
-  )
   (symbol (lib_id "Device:C") (at 109.22 124.46 270) (unit 1)
     (in_bom yes) (on_board yes) (dnp no)
@@
         )
       )
-    )
-  )
-  (symbol (lib_id "Device:R") (at 33.02 95.25 90) (unit 1)
-    (in_bom yes) (on_board yes) (dnp no)
-    (property "Reference" "R2" (at 33.02 92.71 90)
-      (effects (font (size 1.27 1.27)))
-    )
-    (property "Value" "1K" (at 33.02 97.79 90)
-      (effects (font (size 1.27 1.27)))
-    )
-    (property "Footprint" "Resistor_SMD:R_0603_1608Metric_Pad0.98x0.95mm_HandSolder" (at 33.02 97.028 90)
-      (effects (font (size 1.27 1.27)) hide)
-    )
-    (property "Datasheet" "~" (at 33.02 95.25 0)
-      (effects (font (size 1.27 1.27)) hide)
-    )
-    (pin "1")
-    (pin "2")
-    (instances
-      (project "RAK proto board"
-        (path "/320cfaa9-598b-4438-8ba0-f401c00f1f04"
-          (reference "R2") (unit 1)
-        )
-      )

Commit message: Ordered v1.0 on JLCPCB
Parts:
- removed C3: 100nF, Capacitor_Tantalum_SMD:CP_EIA-1608-08_AVX-J, symbol Device:C
- removed J2: UART2 AT, Grove 4 Pins:Grove 4 Pins, symbol Connector_Generic:Conn_01x04
- removed J3: UART1, Grove 4 Pins:Grove 4 Pins, symbol Connector_Generic:Conn_01x04
- removed J4: Groove AIN0 AIN1, Grove 4 Pins:Grove 4 Pins, symbol Connector_Generic:Conn_01x04
- removed J5: Groove AIN2 AIN3, Grove 4 Pins:Grove 4 Pins, symbol Connector_Generic:Conn_01x04
- removed J6: I2C, Grove 4 Pins:Grove 4 Pins, symbol Connector_Generic:Conn_01x04
- removed R6: 10K, Resistor_SMD:R_0603_1608Metric_Pad0.98x0.95mm_HandSolder, symbol Device:R
- removed R8: 0, Resistor_SMD:R_0603_1608Metric_Pad0.98x0.95mm_HandSolder, symbol Device:R
- removed U2: ADS1115IDGS, Package_SO:TSSOP-10_3x3mm_P0.5mm, symbol Analog_ADC:ADS1115IDGS
- added A1/A2: Groove A1 A2, Connector_JST:JST_PH_B4B-PH-K_1x04_P2.00mm_Vertical, symbol Connector_Generic:Conn_01x04
- added A3/A4: Groove A3 A4, Connector_JST:JST_PH_B4B-PH-K_1x04_P2.00mm_Vertical, symbol Connector_Generic:Conn_01x04
- added BOOT0: SW BOOT0, Button_Switch_SMD:SW_Push_1P1T_NO_CK_KMR2, symbol Switch:SW_SPST
- added C12: 1uF, Capacitor_Tantalum_SMD:CP_EIA-1608-08_AVX-J, symbol Device:C
- added C13: 0, Capacitor_Tantalum_SMD:CP_EIA-1608-08_AVX-J, symbol Device:C
- added DIGITAL1: DIGITAL, Connector_JST:JST_PH_B4B-PH-K_1x04_P2.00mm_Vertical, symbol Connector_Generic:Conn_01x04
- added I2C1: I2C, Connector_JST:JST_PH_B4B-PH-K_1x04_P2.00mm_Vertical, symbol Connector_Generic:Conn_01x04
- added R10, R11: 0, Resistor_SMD:R_0603_1608Metric_Pad0.98x0.95mm_HandSolder, symbol Device:R
- added UART1: UART1, Connector_JST:JST_PH_B4B-PH-K_1x04_P2.00mm_Vertical, symbol Connector_Generic:Conn_01x04
- added UART2: UART2 AT, Connector_JST:JST_PH_B4B-PH-K_1x04_P2.00mm_Vertical, symbol Connector_Generic:Conn_01x04
- R9: value 0 -> 10K
- renumbered J7 to BATTERY1, U3 to BME680, C8 to C10, C9 to C11, C11 to C3, C12 to C4, C10 to C5, C5 to C6, C6 to C7, C4 to C8, C7 to C9, J1 to JTAG1, Q1 to KPS-3227, U4 to LIS2DH12, R11 to R2, R12 to R3, R10 to R4, R3 to R5, R4 to R6, R5 to R7, R7 to R8, U1 to RAK3172, SW1 to RST1
Connections:
- net AIN1 is gone; now on net A1: C10.1, C6.2
- net AIN2 is gone; now on net A2: C11.2, C9.2
- net AIN3 is gone; now on net A3: C11.1, C7.2
- net +3V3: now also BOOT0.1 (A), C12.2, DIGITAL1.3 (Pin_3), I2C1.2 (Pin_2), UART1.3 (Pin_3), UART2.3 (Pin_3)
- net A0: now also C10.2, C8.2, A1/A2.4 (Pin_4)
- net A1: now also A1/A2.2 (Pin_2)
- net A2: now also A3/A4.4 (Pin_4)
- net A3: now also A3/A4.2 (Pin_2)
- net A4: now also C5.2, KPS-3227.2, KPS-3227.4, R8.2
- net D0: now also LIS2DH12.11 (INT_2)
- net D1: now also DIGITAL1.1 (Pin_1); no longer D1.1 (K)
- net D2: now also DIGITAL1.2 (Pin_2)
- net D3: now also D1.1 (K)
- net D5: now also LIS2DH12.12 (INT_1)
- net GND: now also R9.1, A1/A2.1 (Pin_1), A1/A2.3 (Pin_3), A3/A4.1 (Pin_1), A3/A4.3 (Pin_3), C12.1, C13.1, DIGITAL1.4 (Pin_4), I2C1.1 (Pin_1), R11.1, UART1.4 (Pin_4), UART2.4 (Pin_4); no longer RAK3172.21 (BOOT0)
- net RF: now also R10.1
- net RX1: now also UART1.1 (Pin_1)
- net RX2: now also UART2.1 (Pin_1)
- net SCL: now also I2C1.4 (Pin_4)
- net SDA: now also I2C1.3 (Pin_3)
- net TX1: now also UART1.2 (Pin_2)
- net TX2: now also UART2.2 (Pin_2)
- removed net AIN0: C10.2, C8.2, R9.1
- new net: C13.2, R10.2, R11.2
- new net BOOT0: BOOT0.2 (B), R9.2, RAK3172.21 (BOOT0)
Other:
- moved on the sheet: C1, C10, C11, C2, C5, C6, C7, C8, C9, D1, KPS-3227, R1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
