File: kicad/mikrobus_x2_hat/mikrobus_x2_hatPCB/mikrobus_x2_hatPCB.kicad_sch (KiCad schematic)
At the start: 3 parts, among them IC1 MIKROE-924, IC2 MIKROE-924, J1 RPi_GPIO

Commit message: Component footprints
Parts:
- added IC3: MCP3204-CI_P, DIP781W56P254L1918H533Q14N, symbol MCP3204:MCP3204-CI_P
- added IC4: TXB0106PWR, SOP65P640X120-16N, symbol TXB0106:TXB0106PWR
- added S1: CAS-D20TA, CAS-D20TA:SW_CAS-D20TA, symbol CAS-D20TA:CAS-D20TA
- added U1: MCP1541, MCP1541:MCP1541, symbol MCP1541:MCP1541

Commit message: PCB completed
Parts:
- removed IC3: MCP3204-CI_P, DIP781W56P254L1918H533Q14N, symbol MCP3204:MCP3204-CI_P
- removed IC4: TXB0106PWR, SOP65P640X120-16N, symbol TXB0106:TXB0106PWR
- removed S1: CAS-D20TA, CAS-D20TA:SW_CAS-D20TA, symbol CAS-D20TA:CAS-D20TA
- removed U1: MCP1541, MCP1541:MCP1541, symbol MCP1541:MCP1541
Connections:
- net at IC1.1 (AN): now also J1.7 (BCM4_GPCLK0)
- net at IC1.10 (INT): now also J1.31 (BCM6)
- net at IC1.11 (RX): now also IC2.11 (RX), J1.10 (BCM15_RXD)
- net at IC1.12 (TX): now also IC2.12 (TX), J1.8 (BCM14_TXD)
- net at IC1.13 (SCL): now also IC2.13 (SCL), J1.5 (BCM3_SCL)
- net at IC1.14 (SDA): now also IC2.14 (SDA), J1.3 (BCM2_SDA)
- net 5V: now reaches IC1.15 (+5V)
- net 5V: now also IC2.15 (+5V), J1.2 (5V), J1.4 (5V)
- net GND: now reaches IC1.16 (GND_2)
- net GND: now also IC1.8 (GND_1), IC2.16 (GND_2), IC2.8 (GND_1), J1.14 (GND), J1.20 (GND), J1.25 (GND), J1.30 (GND), J1.34 (GND), J1.39 (GND), J1.6 (GND), J1.9 (GND)
- net at IC1.2 (RST): now also J1.29 (BCM5)
- net at IC1.3 (CS): now also J1.24 (BCM8_CE0)
- net at IC1.4 (SCK): now also IC2.4 (SCK), J1.23 (BCM11_SCLK)
- net at IC1.5 (MISO): now also IC2.5 (MISO), J1.21 (BCM9_MISO)
- net at IC1.6 (MOSI): now also IC2.6 (MOSI), J1.19 (BCM10_MOSI)
- net 3V3: now reaches IC1.7 (+3.3V)
- net 3V3: now also IC2.7 (+3.3V), J1.1 (3.3V), J1.17 (3.3V)
- net at IC1.9 (PWM): now also J1.12 (BCM18_PCM_C)
- net at J1.11 (BCM17): now also IC2.9 (PWM)
- net at J1.26 (BCM7_CE1): now also IC2.3 (CS)
- net at J1.33 (BCM13_PWM1): now also IC2.1 (AN)
- net at J1.35 (BCM19_MISO_PCM_FS): now also IC2.2 (RST)
- net at J1.37 (BCM26): now also IC2.10 (INT)
- no-connect marks 0 -> 11

Commit message: fix serigraphy
Other:
- title: (none) -> Mikrobus Pi Hat x2
Changed lines of the file:
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@@
 	(generator_version "8.0")
 	(paper "A4")
+	(title_block
+		(title "Mikrobus Pi Hat x2")
+		(date "2024-09-03")
+		(rev "v1.1")
+	)
 	(junction
 		(at 120.65 142.24)

Commit message: reprise schematique, clarification
Parts:
- added JP1, JP2: Jumper_3_Bridged12, Connector_PinSocket_2.54mm:PinSocket_1x03_P2.54mm_Vertical, symbol Jumper:Jumper_3_Bridged12
- IC1, IC2: footprint MIKROE924 -> MIKROE-924:MIKROE924
- J1: footprint (none) -> Connector_PinSocket_2.54mm:PinSocket_2x20_P2.54mm_Vertical
Connections:
- net PWM2: now reaches IC2.9 (PWM), J1.11 (BCM17)
- net PWM1: now reaches IC1.9 (PWM), J1.12 (BCM18_PCM_C)
- net MOSI: now reaches IC1.6 (MOSI), IC2.6 (MOSI), J1.19 (BCM10_MOSI)
- net MISO: now reaches IC1.5 (MISO), IC2.5 (MISO), J1.21 (BCM9_MISO)
- net SCLK: now reaches IC1.4 (SCK), IC2.4 (SCK), J1.23 (BCM11_SCLK)
- net CS1: now reaches IC1.3 (CS), J1.24 (BCM8_CE0)
- net CS2: now reaches IC2.3 (CS), J1.26 (BCM7_CE1)
- net RST1: now reaches IC1.2 (RST), J1.29 (BCM5)
- net SDA: now reaches IC1.14 (SDA), IC2.14 (SDA), J1.3 (BCM2_SDA)
- net INT1: now reaches IC1.10 (INT), J1.31 (BCM6)
- net AN2: now reaches IC2.1 (AN), J1.33 (BCM13_PWM1)
- net RST2: now reaches IC2.2 (RST), J1.35 (BCM19_MISO_PCM_FS)
- net INT2: now reaches IC2.10 (INT), J1.37 (BCM26)
- net SCL: now reaches IC1.13 (SCL), IC2.13 (SCL), J1.5 (BCM3_SCL)
- net AN1: now reaches IC1.1 (AN), J1.7 (BCM4_GPCLK0)
- new net: J1.10 (BCM15_RXD), JP2.2 (C)
- new net: J1.8 (BCM14_TXD), JP1.2 (C)
- new net RX1: IC1.12 (TX), JP2.1 (A)
- new net RX2: IC2.12 (TX), JP2.3 (B)
- new net TX1: IC1.11 (RX), JP1.1 (A)
- new net TX2: IC2.11 (RX), JP1.3 (B)
Other:
- note added: "Mikrobus 1"
- note added: "Mikrobus 2"

Commit message: final commit
Parts:
- IC1, IC2: footprint MIKROE-924:MIKROE924 -> footprint:MIKROE924
- JP1, JP2: footprint Connector_PinSocket_2.54mm:PinSocket_1x03_P2.54mm_Vertical -> Connector_PinHeader_2.54mm:PinHeader_1x03_P2.54mm_Vertical
Changed lines of the file:
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@@
 			)
 		)
-		(property "Footprint" "Connector_PinSocket_2.54mm:PinSocket_1x03_P2.54mm_Vertical"
+		(property "Footprint" "Connector_PinHeader_2.54mm:PinHeader_1x03_P2.54mm_Vertical"
 			(at 207.01 63.5 0)
 			(effects
@@
 			)
 		)
-		(property "Footprint" "Connector_PinSocket_2.54mm:PinSocket_1x03_P2.54mm_Vertical"
+		(property "Footprint" "Connector_PinHeader_2.54mm:PinHeader_1x03_P2.54mm_Vertical"
 			(at 184.15 63.5 0)
 			(effects
@@
 			)
 		)
-		(property "Footprint" "MIKROE-924:MIKROE924"
+		(property "Footprint" "footprint:MIKROE924"
 			(at 229.87 85.09 0)
 			(effects
@@
 			)
 		)
-		(property "Footprint" "MIKROE-924:MIKROE924"
+		(property "Footprint" "footprint:MIKROE924"
 			(at 85.09 86.36 0)
 			(effects
